Commit message: Add obstacles world

File: description/robot_core.xacro (robot description, xacro)
@@ -40,5 +40,5 @@
     </link>
     <gazebo reference="chassis">
-    <material>Gazebo/White</material>
+    <material>Gazebo/Orange</material>
     </gazebo>
     <!-- LEFT WHEEL -->

Commit message: Added mapping in gazebo

File: description/robot_core.xacro (robot description, xacro)
@@ -15,4 +15,12 @@
     </material>
     <link name="base_link">
+    </link>
+    <!-- BASE_FOOTPRINT LINK -->
+    <joint name="base_footprint_joint" type="fixed">
+        <parent link="base_link"/>
+        <child link="base_footprint"/>
+        <origin xyz="0 0 0" rpy="0 0 0"/>
+    </joint>
+    <link name="base_footprint">
     </link>
     <joint name="chassis_joint" type="fixed">
